File: kicad/kicad-c128-byte-wide-color-ram.kicad_sch (KiCad schematic)
At the start: 7 parts, among them J1 A11_A14, J2 AEC, J3 D4_D7, U1 2016-board, U2 KM62256CLP, U3 2016, U4 4066

Commit message: revision 1.1 with 1571CR info
Other:
- note added: "Bytewide Color RAM 2K or 32K Idea: http://www.sdiy.org/richardc64/color/byte.html - install 24 round pins to mainboard in U1 footprint - install socket in U3 (24 pins) for 2K SRAM or U2 (28 pins) for 32K SRAM - install U4 (4066) - connect AEC from onboard U20 (4066) pins 5, 6, 12 or 13 - connect D4-D7_bus in any order from charset ROM nearby (different pinout for 24 and 28 pin chips) - (32K) conn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"
- note added: "ColorRAM: pins to mainboard 1571CR: unpopulated"
- note added: "ColorRAM: socket for 2K SRAM (install only one: for 2K or 32K) 1571CR: pins to mainboard"
- note added: "socket for 32K RAM ColorRAM: install 2K or 32K socket 1571CR: install 32K socket"
- note removed: "AEC and D4_D7 from CPU or VIC"
- note removed: "Idea: http://www.sdiy.org/richardc64/color/byte.html"
- note removed: "pins to mainboard"
- note removed: "socket for 2K SRAM (install one or the other)"
- note removed: "socket for 32K RAM (install one or the other)"
- title: C128 bytewide 2/32K Color RAM -> C128 bytewide 2/32K Color RAM / 1571CR RAM expansion
- moved on the sheet: U4A, U4B, U4C, U4D, U4E
